Commit message: [ros2_control_demo_robot] Fix indentation for rrbot/rrbot_quadruped.urdf.xacro

File: ros2_control_demo_robot/description/rrbot/rrbot_quadruped.urdf.xacro (robot description, xacro)
@@ -18,8 +18,5 @@
         <mass value="1.43315091"/>
         <!-- The base is extremely symmetrical. -->
-        <inertia ixx="0.00578574" ixy="0.0" ixz="0.0"
-                                  iyy="0.01938108" iyz="0.0"
-                                                   izz="0.02476124"
-        />
+        <inertia ixx="0.00578574" ixy="0.0" ixz="0.0" iyy="0.01938108" iyz="0.0" izz="0.02476124" />
     </inertial>
     <!-- BASE LINK VISUAL -->
