Commit message: Add files for seeing the quadruped on rviz2

File: ros2_control_demo_robot/description/rrbot/leg.xacro (robot description, xacro)
@@ -51,5 +51,5 @@
                     <origin xyz="0.01950 0 0" rpy="0 0 0" />
                     <geometry>
-                        <mesh filename="package://robot_properties_solo/meshes/${mesh_ext}/solo12/solo12_hip_fe_fl.${mesh_ext}"/>
+                        <mesh filename="package://ros2_control_demo_robot/description/rrbot/meshes/${mesh_ext}/solo12/solo12_hip_fe_fl.${mesh_ext}"/>
                     </geometry>
                 </xacro:if>
@@ -57,5 +57,5 @@
                     <origin xyz="-0.01950 0 0" rpy="0 0 0" />
                     <geometry>
-                        <mesh filename="package://robot_properties_solo/meshes/${mesh_ext}/solo12/solo12_hip_fe_hl.${mesh_ext}"/>
+                        <mesh filename="package://ros2_control_demo_robot/description/rrbot/meshes/${mesh_ext}/solo12/solo12_hip_fe_hl.${mesh_ext}"/>
                     </geometry>
                 </xacro:unless>
@@ -65,5 +65,5 @@
                     <origin xyz="0.01950 0 0" rpy="0 0 0" />
                     <geometry>
-                        <mesh filename="package://robot_properties_solo/meshes/${mesh_ext}/solo12/solo12_hip_fe_fr.${mesh_ext}"/>
+                        <mesh filename="package://ros2_control_demo_robot/description/rrbot/meshes/${mesh_ext}/solo12/solo12_hip_fe_fr.${mesh_ext}"/>
                     </geometry>
                 </xacro:if>
@@ -71,5 +71,5 @@
                     <origin xyz="-0.01950 0 0" rpy="0 0 0" />
                     <geometry>
-                        <mesh filename="package://robot_properties_solo/meshes/${mesh_ext}/solo12/solo12_hip_fe_hr.${mesh_ext}"/>
+                        <mesh filename="package://ros2_control_demo_robot/description/rrbot/meshes/${mesh_ext}/solo12/solo12_hip_fe_hr.${mesh_ext}"/>
                     </geometry>
                 </xacro:unless>
@@ -85,5 +85,5 @@
                     <origin xyz="0.01950 0 0" rpy="0 0 0" />
                     <geometry>
-                        <mesh filename="package://robot_properties_solo/meshes/${mesh_ext}/solo12/solo12_hip_fe_fl.${mesh_ext}"/>
+                        <mesh filename="package://ros2_control_demo_robot/description/rrbot/meshes/${mesh_ext}/solo12/solo12_hip_fe_fl.${mesh_ext}"/>
                     </geometry>
                 </xacro:if>
@@ -91,5 +91,5 @@
                     <origin xyz="-0.01950 0 0" rpy="0 0 0" />
                     <geometry>
-                        <mesh filename="package://robot_properties_solo/meshes/${mesh_ext}/solo12/solo12_hip_fe_hl.${mesh_ext}"/>
+                        <mesh filename="package://ros2_control_demo_robot/description/rrbot/meshes/${mesh_ext}/solo12/solo12_hip_fe_hl.${mesh_ext}"/>
                     </geometry>
                 </xacro:unless>
@@ -99,5 +99,5 @@
                     <origin xyz="0.01950 0 0" rpy="0 0 0" />
                     <geometry>
-                        <mesh filename="package://robot_properties_solo/meshes/${mesh_ext}/solo12/solo12_hip_fe_fr.${mesh_ext}"/>
+                        <mesh filename="package://ros2_control_demo_robot/description/rrbot/meshes/${mesh_ext}/solo12/solo12_hip_fe_fr.${mesh_ext}"/>
                     </geometry>
                 </xacro:if>
@@ -105,5 +105,5 @@
                     <origin xyz="-0.01950 0 0" rpy="0 0 0" />
                     <geometry>
-                        <mesh filename="package://robot_properties_solo/meshes/${mesh_ext}/solo12/solo12_hip_fe_hr.${mesh_ext}"/>
+                        <mesh filename="package://ros2_control_demo_robot/description/rrbot/meshes/${mesh_ext}/solo12/solo12_hip_fe_hr.${mesh_ext}"/>
                     </geometry>
                 </xacro:unless>
@@ -222,8 +222,8 @@
         <geometry>
           <xacro:unless value="${is_right}">
-            <mesh filename="package://robot_properties_solo/meshes/${mesh_ext}/with_foot/solo_upper_leg_left_side.${mesh_ext}"/>
-          </xacro:unless>
-          <xacro:if value="${is_right}">
-            <mesh filename="package://robot_properties_solo/meshes/${mesh_ext}/with_foot/solo_upper_leg_right_side.${mesh_ext}"/>
+            <mesh filename="package://ros2_control_demo_robot/description/rrbot/meshes/${mesh_ext}/with_foot/solo_upper_leg_left_side.${mesh_ext}"/>
+          </xacro:unless>
+          <xacro:if value="${is_right}">
+            <mesh filename="package://ros2_control_demo_robot/description/rrbot/meshes/${mesh_ext}/with_foot/solo_upper_leg_right_side.${mesh_ext}"/>
           </xacro:if>
         </geometry>
@@ -237,8 +237,8 @@
         <geometry>
           <xacro:unless value="${is_right}">
-            <mesh filename="package://robot_properties_solo/meshes/${mesh_ext}/with_foot/solo_upper_leg_left_side.${mesh_ext}"/>
-          </xacro:unless>
-          <xacro:if value="${is_right}">
-            <mesh filename="package://robot_properties_solo/meshes/${mesh_ext}/with_foot/solo_upper_leg_right_side.${mesh_ext}"/>
+            <mesh filename="package://ros2_control_demo_robot/description/rrbot/meshes/${mesh_ext}/with_foot/solo_upper_leg_left_side.${mesh_ext}"/>
+          </xacro:unless>
+          <xacro:if value="${is_right}">
+            <mesh filename="package://ros2_control_demo_robot/description/rrbot/meshes/${mesh_ext}/with_foot/solo_upper_leg_right_side.${mesh_ext}"/>
           </xacro:if>
         </geometry>
@@ -307,8 +307,8 @@
         <geometry>
           <xacro:unless value="${is_right}">
-            <mesh filename="package://robot_properties_solo/meshes/${mesh_ext}/with_foot/solo_lower_leg_left_side.${mesh_ext}"/>
-          </xacro:unless>
-          <xacro:if value="${is_right}">
-            <mesh filename="package://robot_properties_solo/meshes/${mesh_ext}/with_foot/solo_lower_leg_right_side.${mesh_ext}"/>
+            <mesh filename="package://ros2_control_demo_robot/description/rrbot/meshes/${mesh_ext}/with_foot/solo_lower_leg_left_side.${mesh_ext}"/>
+          </xacro:unless>
+          <xacro:if value="${is_right}">
+            <mesh filename="package://ros2_control_demo_robot/description/rrbot/meshes/${mesh_ext}/with_foot/solo_lower_leg_right_side.${mesh_ext}"/>
           </xacro:if>
         </geometry>
@@ -322,8 +322,8 @@
         <geometry>
           <xacro:unless value="${is_right}">
-            <mesh filename="package://robot_properties_solo/meshes/${mesh_ext}/with_foot/solo_lower_leg_left_side.${mesh_ext}"/>
-          </xacro:unless>
-          <xacro:if value="${is_right}">
-            <mesh filename="package://robot_properties_solo/meshes/${mesh_ext}/with_foot/solo_lower_leg_right_side.${mesh_ext}"/>
+            <mesh filename="package://ros2_control_demo_robot/description/rrbot/meshes/${mesh_ext}/with_foot/solo_lower_leg_left_side.${mesh_ext}"/>
+          </xacro:unless>
+          <xacro:if value="${is_right}">
+            <mesh filename="package://ros2_control_demo_robot/description/rrbot/meshes/${mesh_ext}/with_foot/solo_lower_leg_right_side.${mesh_ext}"/>
           </xacro:if>
         </geometry>
@@ -368,5 +368,5 @@
         <origin xyz="0 0 0" rpy="0 0 0" />
         <geometry>
-          <mesh filename="package://robot_properties_solo/meshes/${mesh_ext}/with_foot/solo_foot.${mesh_ext}"/>
+          <mesh filename="package://ros2_control_demo_robot/description/rrbot/meshes/${mesh_ext}/with_foot/solo_foot.${mesh_ext}"/>
         </geometry>
         <material name="${color_name}">
@@ -378,5 +378,5 @@
         <origin xyz="0 0 0" rpy="0 0 0" />
         <geometry>
-            <mesh filename="package://robot_properties_solo/meshes/${mesh_ext}/with_foot/solo_foot.${mesh_ext}"/>
+            <mesh filename="package://ros2_control_demo_robot/description/rrbot/meshes/${mesh_ext}/with_foot/solo_foot.${mesh_ext}"/>
         </geometry>
         <material name="${color_name}">

File: ros2_control_demo_robot/description/rrbot/rrbot_quadruped.urdf.xacro (robot description, xacro)
@@ -24,5 +24,5 @@
         <origin xyz="0 0 0" rpy="0 0 0" />
         <geometry>
-          <mesh filename="package://ros2_control_demo_robot/description/meshes/${mesh_ext}/with_foot/solo_body.${mesh_ext}"/>
+          <mesh filename="package://ros2_control_demo_robot/description/rrbot/meshes/${mesh_ext}/with_foot/solo_body.${mesh_ext}"/>
         </geometry>
         <material name="${color_name}">
